File: milkyway.kicad_pcb (KiCad board)
At the start: 2 copper layers, 304.4 x 98.8 mm, 162 parts, among them J10 Conn_01x01, J11 Conn_01x01, J12 Conn_01x01, J13 Conn_01x01, J14 Conn_01x01, J15 Conn_01x01, J16 Conn_01x01, J17 Conn_01x01, J8 Conn_01x01, J9 Conn_01x01, SW0 SW_PUSH, U1 Raspberry_Pi_Pico

Commit message: さらに追加調整
Parts:
- moved SWR17 2.38 mm to (309.6, 47.6)
- moved DR07 1.27 mm to (304.8, 39.4)
- moved DR04 0.61 mm to (190.5, 33.3)
- moved DC42 0.13 mm to (206.0, 109.6)
- moved DR43 0.13 mm to (208.5, 109.6)
- moved DR46 0.13 mm to (295.1, 109.5)
Routing:
- net Col3: track 355.0 -> 376.1 mm, vias 7 -> 11
- net Col1: track 443.6 -> 463.2 mm
- net Col2: track 428.2 -> 446.5 mm, vias 8 -> 5
- net Col0: track 504.7 -> 521.9 mm
- net Row3: track 441.7 -> 429.0 mm, vias 3 -> 1
- net Col6: track 284.6 -> 296.7 mm
- net Col4: track 254.4 -> 263.6 mm, vias 5 -> 10
- net Row0: track 405.6 -> 396.5 mm
- net Col5: track 257.4 -> 266.3 mm, vias 6 -> 10
- net Col7: track 116.3 -> 124.6 mm
- net Net-(DR36-Pad1): track 45.2 -> 51.9 mm
- net Row2: track 373.7 -> 367.3 mm
- net Row1: track 379.8 -> 373.5 mm
- net Rot5B: track 192.4 -> 196.2 mm, vias 4 -> 0
- net Rot4A: track 146.6 -> 150.1 mm, vias 4 -> 0
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