File: milkyway.kicad_pcb (KiCad board)
At the start: 2 copper layers, 304.4 x 98.8 mm, 162 parts, among them J10 Conn_01x01, J11 Conn_01x01, J12 Conn_01x01, J13 Conn_01x01, J14 Conn_01x01, J15 Conn_01x01, J16 Conn_01x01, J17 Conn_01x01, J8 Conn_01x01, J9 Conn_01x01, SW0 SW_PUSH, U1 Raspberry_Pi_Pico

Commit message: 組み立て補助のためのシルク調整
Parts:
- added G***: LOGO, milkyway:Raspberry_Pi_Logo, B.Cu at (233.0, 37.5)
Routing:
- net Rot4A: track 150.1 -> 146.1 mm
- net Rot4B: track 164.4 -> 160.5 mm
- net Col3: track 376.1 -> 373.5 mm
- net GND: track 377.1 -> 379.0 mm
- net Col0: track 521.9 -> 522.4 mm
Other:
- board text added: "2"
- board text added: "3"
- board text added: "4"
- board text added: "A"
- board text added: "B"
- board text added: "C"
- board text added: "D"
- board text added: "↙1↘"
- board text added: "↙5↘"

Commit message: image directory. design logo on back. front soon.
Parts:
- added G***: LOGO, milkyway:Silk_Special_Thanks, B.Cu at (95.2, 20.7)
- added G***: LOGO, milkyway:Silk_Author, B.Cu at (191.9, 20.7)

Commit message: front silk design
Parts:
- added G***: LOGO, milkyway:Silk_Title, F.Cu at (94.7, 52.6)
- added G***: LOGO, milkyway:Silk_Title_Sub, F.Cu at (140.7, 138.6)
- moved G*** 20.1 mm to (184.4, 39.4)
- moved G*** 19.3 mm to (99.4, 39.5)
Routing:
- net Net-(DR33-Pad1): track 23.4 -> 22.6 mm
Other:
- board text added: "for GL516"

Commit message: 微修正
Parts:
- removed the G*** at (140.7, 138.6)
